Commit message: fix

File: dist/gripper.urdf (robot description, URDF)
Before this commit: robot gripper, 10 links, 9 joints
Links:
- link cam: geometry collision mesh filename=assets/cam.stl; visual mesh filename=assets/cam.stl
- link distal_shell: geometry collision mesh filename=assets/distal_rod.stl; collision mesh filename=assets/distal_shell.stl
- link distal_shell_2: geometry collision mesh filename=assets/distal_rod.stl; collision mesh filename=assets/distal_shell.stl
- link external_rod: geometry collision mesh filename=assets/external_rod.stl; visual mesh filename=assets/external_rod.stl
- link external_rod_2: geometry collision mesh filename=assets/external_rod.stl; visual mesh filename=assets/external_rod.stl
- link interface_arm100: geometry collision mesh filename=assets/bottom_plate.stl; collision mesh filename=assets/camera_basement.stl
- link internal_rod: geometry collision mesh filename=assets/internal_rod.stl; visual mesh filename=assets/internal_rod.stl
- link internal_rod_2: geometry collision mesh filename=assets/internal_rod.stl; visual mesh filename=assets/internal_rod.stl

File: dist/robot.urdf (robot description, URDF)
Before this commit: robot robot, 8 links, 7 joints
Links:
- link base_so101_v2: geometry collision mesh filename=assets/base_motor_holder_so101_v1.stl; collision mesh filename=assets/base_so101_v2.stl
- link component1___use: geometry collision mesh filename=assets/component1___use.stl; collision mesh filename=assets/motor_holder_so101_wrist_v1.stl
- link rotation_pitch_so101_v1: geometry collision mesh filename=assets/motor_holder_so101_base_v1.stl; collision mesh filename=assets/rotation_pitch_so101_v1.stl
- link sts3215_03a_v1: geometry collision mesh filename=assets/sts3215_03a_v1.stl; collision mesh filename=assets/wrist_roll_pitch_so101_v2.stl
- link upper_arm_so101_v1: geometry collision mesh filename=assets/sts3215_03a_v1__3.stl; collision mesh filename=assets/upper_arm_so101_v1.stl
- link wrist_roll_pitch_so101_v2: geometry collision mesh filename=assets/sts3215_03a_v1__3.stl; collision mesh filename=assets/wrist_roll_pitch_so101_v2.stl

File: dist/xlerobot.urdf (robot description, URDF)
Before this commit: robot urdf_xlerobot, 4 links, 3 joints
Links:
- link 035armbase_step: geometry collision mesh filename=assets/035armbase_step.stl; collision mesh filename=assets/035armbase_step__2.stl
